Commit message: Humble build (#52)
* Fix templates on declaring parameters

* Fix runtime errors

* Update noether for humble build

* add vtk to rosdep skip

* Updated dependencies to be by ROS version

* Change skip key to just 'libvtk'

* Check ROS version for how params are declared

* Added ROS version check for tf2_eigen include

* Added tf2_eigen depends to various packages

* Added tf2_eigen to planning package CMakeLists

* Fixed a templated declare param previously missed

* Clang formatting

* Clang formatting (pt 2)

* Cleaner ROS version checking

* Set C++ version to 17 for `__has_include` macro

* Removed #if's from different ROS versions

* Fix where things built, but didn't work in humble

* Fix load_yaml difference between foxy and humble+

* Clang formatting

* Update snp_blending support to work with humble

File: urdf/workcell.xacro (robot description, xacro)
@@ -130,5 +130,11 @@
     <child link="ee"/>
   </joint>
-  <xacro:property name="camera_cal" value="${load_yaml('$(find snp_automate_2022)/config/camera_calibration.yaml')}" />
+  <xacro:arg name="ros_distro" default="humble"/>
+  <xacro:if value="${'$(arg ros_distro)' > 'foxy'}">
+    <xacro:property name="camera_cal" value="${xacro.load_yaml('$(find snp_automate_2022)/config/camera_calibration.yaml')}" />
+  </xacro:if>
+  <xacro:unless value="${'$(arg ros_distro)' > 'foxy'}">
+    <xacro:property name="camera_cal" value="${load_yaml('$(find snp_automate_2022)/config/camera_calibration.yaml')}" />
+  </xacro:unless>
   <link name="camera_color_optical_frame"/>
   <joint name="tool0_to_camera" type="fixed">

Commit message: Added media geometry to TCP

File: urdf/workcell.xacro (robot description, xacro)
@@ -152,5 +152,21 @@
   </joint>
   <!-- Add TCP -->
-  <link name="sand_tcp"/>
+  <xacro:property name="media_radius" value="0.075"/>
+  <xacro:property name="media_length" value="0.05"/>
+  <xacro:property name="media_collision_offset" value="0.01"/>
+  <link name="sand_tcp">
+    <visual>
+      <origin xyz="0.0 0.0 ${-(media_length / 2.0)}"/>
+      <geometry>
+        <cylinder radius="${media_radius}" length="${media_length}"/>
+      </geometry>
+    </visual>
+    <collision>
+      <origin xyz="0.0 0.0 ${-(media_length / 2.0) - media_collision_offset}"/>
+      <geometry>
+        <cylinder radius="${media_radius}" length="${media_length - media_collision_offset}"/>
+      </geometry>
+    </collision>
+  </link>
   <joint name="sand_tcp_joint" type="fixed">
     <parent link="tool_flange"/>

Commit message: Rotated TCP to accommodate change to SNP motion planner

File: urdf/workcell.xacro (robot description, xacro)
@@ -119,10 +119,4 @@
       </geometry>
     </collision>
-    <collision name="tcp">
-      <geometry>
-        <cylinder radius="${1.5 * 0.0254}" length="${2.0 * 0.0254}"/>
-      </geometry>
-      <origin xyz="${-0.263 + 1.5 * 0.0254} 0.0 0.083" rpy="0 ${radians(-90)} 0"/>
-    </collision>
   </link>
   <joint name="tool0_to_ee" type="fixed">
@@ -157,5 +151,5 @@
   <link name="sand_tcp">
     <visual>
-      <origin xyz="0.0 0.0 ${-(media_length / 2.0)}"/>
+      <origin xyz="0.0 0.0 ${(media_length / 2.0)}"/>
       <geometry>
         <cylinder radius="${media_radius}" length="${media_length}"/>
@@ -163,5 +157,5 @@
     </visual>
     <collision>
-      <origin xyz="0.0 0.0 ${-(media_length / 2.0) - media_collision_offset}"/>
+      <origin xyz="0.0 0.0 ${(media_length / 2.0) + media_collision_offset}"/>
       <geometry>
         <cylinder radius="${media_radius}" length="${media_length - media_collision_offset}"/>
@@ -172,5 +166,5 @@
     <parent link="tool_flange"/>
     <child link="sand_tcp"/>
-    <origin xyz="-0.26261 0 ${0.08259 + dt_flange_width}" rpy="${radians(-90)} 0 ${radians(90)}"/>
+    <origin xyz="-0.26261 0 ${0.08259 + dt_flange_width}" rpy="${radians(90)} 0 ${radians(90)}"/>
   </joint>
 </robot>
